File: kicad/gimbal-board.sch (KiCad schematic (older format))
At the start: 34 parts, among them IC1 ATMEGA328P-A, P1 ICSP_CONN, P2 BAT_CONN, P3 MOTOR_CONN, P4 IMU_CONN, P5 FTDI_CONN, P6 3V3_CONN, SW1 SW_PUSH, SW2 SW_PUSH, U1 DRV10975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

Commit message: Remade Rev 01 layout and sent to fab
Parts:
- removed P1: ICSP_CONN, Pin_Headers:Pin_Header_Straight_2x03, symbol CONN_02X03
- added P1: ICSP, Pin_Headers:Pin_Header_Straight_1x06, symbol CONN_01X06
- P2: value BAT_CONN -> BATT
- P3: value MOTOR_CONN -> MOTOR
- P4: value IMU_CONN -> IMU
- P5: value FTDI_CONN -> FTDI
- gave numbers to parts that had none: 4
Connections:
- net +3V3: now also R6.1, P1.1 (P1)
- net GND: now also P1.6 (P6)
- net ICSP_MISO: now also P1.3 (P3)
- net ICSP_MOSI: now also P1.2 (P2)
- net ICSP_SCK: now also P1.4 (P4)
- net RESET: now also P1.5 (P5)
- net V3P3: no longer R6.1
Other:
- moved on the sheet: P2, P3, R6
Changed lines of the file:
@@
 P 9450 1650
 F 0 "P4" H 9528 1688 50  0000 L CNN
-F 1 "IMU_CONN" H 9528 1596 50  0000 L CNN
+F 1 "IMU" H 9528 1596 50  0000 L CNN
 F 2 "Pin_Headers:Pin_Header_Straight_1x08" H 9450 1650 50  0001 C CNN
 F 3 "" H 9450 1650 50  0000 C CNN
@@
 L CONN_01X02 P2
 U 1 1 56C68556
-P 8050 1800
-F 0 "P2" H 8128 1838 50  0000 L CNN
-F 1 "BAT_CONN" H 8128 1746 50  0000 L CNN
-F 2 "Pin_Headers:Pin_Header_Straight_1x02" H 8050 1800 50  0001 C CNN
-F 3 "" H 8050 1800 50  0000 C CNN
-	1    8050 1800
+P 8050 1350
+F 0 "P2" H 8128 1388 50  0000 L CNN
+F 1 "BATT" H 8128 1296 50  0000 L CNN
+F 2 "Pin_Headers:Pin_Header_Straight_1x02" H 8050 1350 50  0001 C CNN
+F 3 "" H 8050 1350 50  0000 C CNN
+	1    8050 1350
 	-1   0    0    -1
 $EndComp
@@
 L +BATT #PWR011
 U 1 1 56C6877C
-P 8300 1700
-F 0 "#PWR011" H 8300 1550 50  0001 C CNN
-F 1 "+BATT" H 8318 1874 50  0000 C CNN
-F 2 "" H 8300 1700 50  0000 C CNN
-F 3 "" H 8300 1700 50  0000 C CNN
-	1    8300 1700
+P 8300 1250
+F 0 "#PWR011" H 8300 1100 50  0001 C CNN
+F 1 "+BATT" H 8318 1424 50  0000 C CNN
+F 2 "" H 8300 1250 50  0000 C CNN
+F 3 "" H 8300 1250 50  0000 C CNN
+	1    8300 1250
 	-1   0    0    -1
 $EndComp
@@
 L GND #PWR012
 U 1 1 56C687AC
-P 8300 1900
-F 0 "#PWR012" H 8300 1650 50  0001 C CNN
-F 1 "GND" H 8308 1726 50  0000 C CNN
-F 2 "" H 8300 1900 50  0000 C CNN
-F 3 "" H 8300 1900 50  0000 C CNN
-	1    8300 1900
+P 8300 1450
+F 0 "#PWR012" H 8300 1200 50  0001 C CNN
+F 1 "GND" H 8308 1276 50  0000 C CNN
+F 2 "" H 8300 1450 50  0000 C CNN
+F 3 "" H 8300 1450 50  0000 C CNN
+	1    8300 1450
 	-1   0    0    -1
 $EndComp
@@
 L CONN_01X03 P3
 U 1 1 56C68C56
-P 8050 2350
-F 0 "P3" H 8128 2388 50  0000 L CNN
-F 1 "MOTOR_CONN" H 8128 2296 50  0000 L CNN
-F 2 "Pin_Headers:Pin_Header_Straight_1x03" H 8050 2350 50  0001 C CNN
-F 3 "" H 8050 2350 50  0000 C CNN
-	1    8050 2350
-	-1   0    0    -1
-$EndComp
-Text Label 8800 2250 2    60   ~ 0
+P 8050 1900
+F 0 "P3" H 8128 1938 50  0000 L CNN
+F 1 "MOTOR" H 8128 1846 50  0000 L CNN
+F 2 "Pin_Headers:Pin_Header_Straight_1x03" H 8050 1900 50  0001 C CNN
+F 3 "" H 8050 1900 50  0000 C CNN
+	1    8050 1900
+	-1   0    0    -1
+$EndComp
+Text Label 8800 1800 2    60   ~ 0
 M_PHASE_U
-Text Label 8800 2350 2    60   ~ 0
+Text Label 8800 1900 2    60   ~ 0
 M_PHASE_V
-Text Label 8800 2450 2    60   ~ 0
+Text Label 8800 2000 2    60   ~ 0
 M_PHASE_W
 NoConn ~ 9650 1700
@@
 Text Label 4150 3450 2    60   ~ 0
 M_SPEED
-$Comp
-L CONN_02X03 P1
-U 1 1 56C7E224
-P 3150 1950
-F 0 "P1" H 3150 2266 50  0000 C CNN
-F 1 "ICSP_CONN" H 3150 2174 50  0000 C CNN
-F 2 "Pin_Headers:Pin_Header_Straight_2x03" H 3150 750 50  0001 C CNN
-F 3 "" H 3150 750 50  0000 C CNN
-	1    3150 1950
-	1    0    0    -1
-$EndComp
-Text Label 2400 1850 0    60   ~ 0
+Text Label 8550 2600 2    60   ~ 0
 ICSP_MISO
-Text Label 2400 1950 0    60   ~ 0
+Text Label 8550 2700 2    60   ~ 0
 ICSP_SCK
-Text Label 2400 2050 0    60   ~ 0
+Text Label 8550 2800 2    60   ~ 0
 RESET
-Text Label 3900 1950 2    60   ~ 0
+Text Label 8550 2500 2    60   ~ 0
 ICSP_MOSI
 $Comp
 L GND #PWR018
 U 1 1 56C7E7BD
-P 3450 2100
-F 0 "#PWR018" H 3450 1850 50  0001 C CNN
-F 1 "GND" H 3458 1926 50  0000 C CNN
-F 2 "" H 3450 2100 50  0000 C CNN
-F 3 "" H 3450 2100 50  0000 C CNN
-	1    3450 2100
+P 8100 2950
+F 0 "#PWR018" H 8100 2700 50  0001 C CNN
+F 1 "GND" H 8108 2776 50  0000 C CNN
+F 2 "" H 8100 2950 50  0000 C CNN
+F 3 "" H 8100 2950 50  0000 C CNN
+	1    8100 2950
 	1    0    0    -1
 $EndComp
@@
 L +3.3V #PWR019
 U 1 1 56C7E7F7
-P 3450 1800
-F 0 "#PWR019" H 3450 1650 50  0001 C CNN
-F 1 "+3.3V" H 3468 1974 50  0000 C CNN
-F 2 "" H 3450 1800 50  0000 C CNN
-F 3 "" H 3450 1800 50  0000 C CNN
-	1    3450 1800
+P 8100 2350
+F 0 "#PWR019" H 8100 2200 50  0001 C CNN
+F 1 "+3.3V" H 8118 2524 50  0000 C CNN
+F 2 "" H 8100 2350 50  0000 C CNN
+F 3 "" H 8100 2350 50  0000 C CNN
+	1    8100 2350
 	1    0    0    -1
 $EndComp
@@
 L R R6
 U 1 1 56C8DFB4
-P 6200 5450
-F 0 "R6" V 5992 5450 50  0000 C CNN
-F 1 "DNP" V 6084 5450 50  0000 C CNN
-F 2 "Resistors_SMD:R_0805_HandSoldering" V 6130 5450 50  0001 C CNN
-F 3 "" H 6200 5450 50  0000 C CNN
-	1    6200 5450
+P 4650 2500
+F 0 "R6" V 4442 2500 50  0000 C CNN
+F 1 "DNP" V 4534 2500 50  0000 C CNN
+F 2 "Resistors_SMD:R_0805_HandSoldering" V 4580 2500 50  0001 C CNN
+F 3 "" H 4650 2500 50  0000 C CNN
+	1    4650 2500
 	0    1    1    0
 $EndComp
@@
 	0    1    1    0
 $EndComp
-Text Label 6650 5450 2    60   ~ 0
-V3P3
 Wire Wire Line
 	1650 3300 1650 3650
@@
 Connection ~ 1750 1500
 Wire Wire Line
-	8300 1700 8300 1750
-Wire Wire Line
-	8300 1750 8250 1750
-Wire Wire Line
-	8300 1900 8300 1850
-Wire Wire Line
-	8300 1850 8250 1850
-Wire Wire Line
-	8250 2250 8800 2250
-Wire Wire Line
-	8250 2350 8800 2350
-Wire Wire Line
-	8250 2450 8800 2450
+	8300 1250 8300 1300
+Wire Wire Line
+	8300 1300 8250 1300
+Wire Wire Line
+	8300 1450 8300 1400
+Wire Wire Line
+	8300 1400 8250 1400
+Wire Wire Line
+	8250 1800 8800 1800
+Wire Wire Line
+	8250 1900 8800 1900
+Wire Wire Line
+	8250 2000 8800 2000
 Wire Wire Line
 	7350 4400 7400 4400
@@
 	3600 3450 4150 3450
 Wire Wire Line
-	2900 1850 2400 1850
-Wire Wire Line
-	2400 1950 2900 1950
-Wire Wire Line
-	2400 2050 2900 2050
-Wire Wire Line
-	3400 1950 3900 1950
-Wire Wire Line
-	3400 1850 3450 1850
-Wire Wire Line
-	3450 1850 3450 1800
-Wire Wire Line
-	3400 2050 3450 2050
-Wire Wire Line
-	3450 2050 3450 2100
+	8050 2600 8550 2600
+Wire Wire Line
+	8550 2700 8050 2700
+Wire Wire Line
+	8550 2800 8050 2800
+Wire Wire Line
+	8050 2500 8550 2500
+Wire Wire Line
+	8050 2400 8100 2400
+Wire Wire Line
+	8100 2400 8100 2350
+Wire Wire Line
+	8050 2900 8100 2900
+Wire Wire Line
+	8100 2900 8100 2950
 Wire Wire Line
 	3600 4700 4150 4700
@@
 Connection ~ 9200 4400
 Wire Wire Line
-	6350 5450 6650 5450
-Wire Wire Line
 	4850 2150 4800 2150
 Wire Wire Line
 	4800 1800 4850 1800
-Text Label 5800 5450 0    60   ~ 0
+Text Label 4250 2500 0    60   ~ 0
 M_FG
 Text Label 4250 1800 0    60   ~ 0
@@
 SDA
 Wire Wire Line
-	6050 5450 5800 5450
+	4500 2500 4250 2500
 Wire Wire Line
 	4250 1800 4500 1800
@@
 P 9450 2600
 F 0 "P5" H 9600 2700 50  0000 C CNN
-F 1 "FTDI_CONN" H 9750 2600 50  0000 C CNN
+F 1 "FTDI" H 9750 2600 50  0000 C CNN
 F 2 "Pin_Headers:Pin_Header_Straight_1x06" H 9450 2600 50  0001 C CNN
 F 3 "" H 9450 2600 50  0000 C CNN
@@
 	10600 950  10600 3500
 Wire Wire Line
-	4850 1800 4850 2150
+	4850 1800 4850 2500
 $Comp
 L +3.3V #PWR029
@@
 	3600 3350 4150 3350
 $Comp
-L CONN_01X01 H?
+L CONN_01X01 H3
 U 1 1 56CBD08A
 P 1300 7250
-F 0 "H?" H 1377 7334 50  0000 L CNN
+F 0 "H3" H 1377 7334 50  0000 L CNN
 F 1 "CONN_01X01" H 1377 7242 50  0000 L CNN
 F 2 "Mounting_Holes:MountingHole_3mm" H 1377 7150 50  0000 L CNN
@@
 $EndComp
 $Comp
-L CONN_01X01 H?
+L CONN_01X01 H4
 U 1 1 56CBD689
 P 1300 7550
-F 0 "H?" H 1377 7634 50  0000 L CNN
+F 0 "H4" H 1377 7634 50  0000 L CNN
 F 1 "CONN_01X01" H 1377 7542 50  0000 L CNN
 F 2 "Mounting_Holes:MountingHole_3mm" H 1377 7450 50  0000 L CNN
@@
 $EndComp
 $Comp
-L CONN_01X01 H?
+L CONN_01X01 H2
 U 1 1 56CBD6FF
 P 1300 6950
-F 0 "H?" H 1377 7034 50  0000 L CNN
+F 0 "H2" H 1377 7034 50  0000 L CNN
 F 1 "CONN_01X01" H 1377 6942 50  0000 L CNN
 F 2 "Mounting_Holes:MountingHole_3mm" H 1377 6850 50  0000 L CNN
@@
 $EndComp
 $Comp
-L CONN_01X01 H?
+L CONN_01X01 H1
 U 1 1 56CBD778
 P 1300 6650
-F 0 "H?" H 1377 6734 50  0000 L CNN
+F 0 "H1" H 1377 6734 50  0000 L CNN
 F 1 "CONN_01X01" H 1377 6642 50  0000 L CNN
 F 2 "Mounting_Holes:MountingHole_3mm" H 1377 6550 50  0000 L CNN
@@
 NoConn ~ 1100 7250
 NoConn ~ 1100 7550
+$Comp
+L CONN_01X06 P1
+U 1 1 56CB80A9
+P 7850 2650
+F 0 "P1" H 7928 2688 50  0000 L CNN
+F 1 "ICSP" H 7928 2596 50  0000 L CNN
+F 2 "Pin_Headers:Pin_Header_Straight_1x06" H 7928 2550 50  0001 L CNN
+F 3 "" H 7850 2650 50  0000 C CNN
+	1    7850 2650
+	-1   0    0    -1
+$EndComp
+Connection ~ 4850 2150
+Wire Wire Line
+	4850 2500 4800 2500
 $EndSCHEMATC
