File: kicad/r1_gimbal-board.kicad_pcb (KiCad board)
At the start: 2 copper layers, 79 x 45 mm, 34 parts, among them IC1 ATMEGA328P-A, P1 ICSP_CONN, P2 BAT_CONN, P3 MOTOR_CONN, P4 IMU_CONN, P5 FTDI_CONN, P6 3V3_CONN, SW1 SW_PUSH, SW2 SW_PUSH, U1 DRV10975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

Commit message: Remade Rev 01 layout and sent to fab
Changed lines of the file:
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@@
 (kicad_pcb (version 4) (host pcbnew 0.201602181416+6564~42~ubuntu15.04.1-product)
   (general
-    (links 84)
+    (links 83)
     (no_connects 0)
     (area 99.892427 23.8745 181.627381 71.97626)
@@
   )
   (setup
-    (last_trace_width 0.25)
+    (last_trace_width 0.5)
     (user_trace_width 0.5)
     (user_trace_width 0.75)
@@
     (tags "capacitor 0805")
     (attr smd)
-    (fp_text reference C10 (at 3.352527 -0.167363 180) (layer F.SilkS)
+    (fp_text reference C10 (at 0 -2.1 90) (layer F.SilkS)
       (effects (font (size 1 1) (thickness 0.15)))
     )
@@
     (tags "resistor 0805")
     (attr smd)
-    (fp_text reference R2 (at 3.352527 0.232637 180) (layer F.SilkS)
-      (effects (font (size 1 1) (thickness 0.15)))
-    )
+    (fp_text reference R2 (at 0 -2.1 90) (layer F.SilkS)
+      (effects (font (size 1 1) (thickness 0.15)))
+    )
